Commit message: feat: Обновить компактную расчетную модель манипулятора с новыми параметрами и документацией

File: src/arm_description/urdf/arm.urdf.xacro (robot description, xacro)
@@ -4,4 +4,22 @@
          Иначе (MoveIt/mock) интерфейсы объявляет arm.ros2_control.xacro — дублировать нельзя. -->
     <xacro:arg name="use_gazebo" default="false"/>
+    <!-- Компактный прототип с нейтральной высотой TCP около 0.50 м. -->
+    <xacro:property name="base_width" value="0.16"/>
+    <xacro:property name="base_height" value="0.10"/>
+    <xacro:property name="upper_arm_length" value="0.12"/>
+    <xacro:property name="forearm_length" value="0.13"/>
+    <xacro:property name="wrist_mount_length" value="0.08"/>
+    <xacro:property name="wrist_roll_length" value="0.025"/>
+    <xacro:property name="wrist_pitch_length" value="0.02"/>
+    <xacro:property name="tool_flange_length" value="0.02"/>
+    <xacro:property name="tcp_offset" value="0.025"/>
+    <!-- Проектный mass budget модели равен 4.15 кг с учетом основания. -->
+    <xacro:property name="base_mass" value="1.2"/>
+    <xacro:property name="upper_arm_mass" value="0.9"/>
+    <xacro:property name="forearm_mass" value="0.8"/>
+    <xacro:property name="wrist_mount_mass" value="0.45"/>
+    <xacro:property name="wrist_roll_mass" value="0.35"/>
+    <xacro:property name="wrist_pitch_mass" value="0.25"/>
+    <xacro:property name="tool_flange_mass" value="0.2"/>
     <!-- Цвета для RViz -->
     <material name="gray"><color rgba="0.3 0.3 0.3 1.0"/></material>
@@ -20,16 +38,21 @@
     <link name="base_link">
         <visual>
-            <origin xyz="0 0 0.1" rpy="0 0 0"/>
-            <geometry><box size="0.2 0.2 0.2"/></geometry>
+            <origin xyz="0 0 ${base_height / 2}" rpy="0 0 0"/>
+            <geometry><box size="${base_width} ${base_width} ${base_height}"/></geometry>
             <material name="gray"/>
         </visual>
         <collision>
-            <origin xyz="0 0 0.1" rpy="0 0 0"/>
-            <geometry><box size="0.2 0.2 0.2"/></geometry>
-        </collision>
-        <inertial>
-            <origin xyz="0 0 0.1" rpy="0 0 0"/>
-            <mass value="2.0"/>
-            <inertia ixx="0.0133" ixy="0.0" ixz="0.0" iyy="0.0133" iyz="0.0" izz="0.0133"/>
+            <origin xyz="0 0 ${base_height / 2}" rpy="0 0 0"/>
+            <geometry><box size="${base_width} ${base_width} ${base_height}"/></geometry>
+        </collision>
+        <inertial>
+            <origin xyz="0 0 ${base_height / 2}" rpy="0 0 0"/>
+            <mass value="${base_mass}"/>
+            <inertia
+                ixx="${base_mass * (base_width ** 2 + base_height ** 2) / 12}"
+                ixy="0.0" ixz="0.0"
+                iyy="${base_mass * (base_width ** 2 + base_height ** 2) / 12}"
+                iyz="0.0"
+                izz="${base_mass * (2 * base_width ** 2) / 12}"/>
         </inertial>
     </link>
@@ -37,28 +60,33 @@
         <material>Gazebo/Grey</material>
     </gazebo>
-    <!-- JOINT 1: BASE YAW (ось Z), 0.20 -> 0.45 м -->
+    <!-- JOINT 1, вращение основания вокруг Z -->
     <joint name="joint_1" type="revolute">
         <parent link="base_link"/>
         <child link="link_1"/>
-        <origin xyz="0 0 0.2" rpy="0 0 0"/>
+        <origin xyz="0 0 ${base_height}" rpy="0 0 0"/>
         <axis xyz="0 0 1"/>
         <limit lower="-3.14159" upper="3.14159" effort="150.0" velocity="2.0"/>
         <dynamics damping="0.5" friction="0.1"/>
     </joint>
-    <!-- LINK 1 (плечо, 0.25 м) -->
+    <!-- LINK 1, верхнее плечо -->
     <link name="link_1">
         <visual>
-            <origin xyz="0 0 0.125" rpy="0 0 0"/>
-            <geometry><cylinder length="0.25" radius="0.06"/></geometry>
+            <origin xyz="0 0 ${upper_arm_length / 2}" rpy="0 0 0"/>
+            <geometry><cylinder length="${upper_arm_length}" radius="0.035"/></geometry>
             <material name="blue"/>
         </visual>
         <collision>
-            <origin xyz="0 0 0.125" rpy="0 0 0"/>
-            <geometry><cylinder length="0.25" radius="0.06"/></geometry>
-        </collision>
-        <inertial>
-            <origin xyz="0 0 0.125" rpy="0 0 0"/>
-            <mass value="1.8"/>
-            <inertia ixx="0.0110" ixy="0.0" ixz="0.0" iyy="0.0110" iyz="0.0" izz="0.00324"/>
+            <origin xyz="0 0 ${upper_arm_length / 2}" rpy="0 0 0"/>
+            <geometry><cylinder length="${upper_arm_length}" radius="0.035"/></geometry>
+        </collision>
+        <inertial>
+            <origin xyz="0 0 ${upper_arm_length / 2}" rpy="0 0 0"/>
+            <mass value="${upper_arm_mass}"/>
+            <inertia
+                ixx="${upper_arm_mass * (3 * 0.035 ** 2 + upper_arm_length ** 2) / 12}"
+                ixy="0.0" ixz="0.0"
+                iyy="${upper_arm_mass * (3 * 0.035 ** 2 + upper_arm_length ** 2) / 12}"
+                iyz="0.0"
+                izz="${upper_arm_mass * 0.035 ** 2 / 2}"/>
         </inertial>
     </link>
@@ -66,28 +94,33 @@
         <material>Gazebo/Blue</material>
     </gazebo>
-    <!-- JOINT 2: SHOULDER PITCH (ось Y), 0.45 -> 0.75 м -->
+    <!-- JOINT 2, наклон плеча вокруг Y -->
     <joint name="joint_2" type="revolute">
         <parent link="link_1"/>
         <child link="link_2"/>
-        <origin xyz="0 0 0.25" rpy="0 0 0"/>
+        <origin xyz="0 0 ${upper_arm_length}" rpy="0 0 0"/>
         <axis xyz="0 1 0"/>
         <limit lower="-2.0944" upper="2.0944" effort="150.0" velocity="2.0"/>
         <dynamics damping="0.5" friction="0.1"/>
     </joint>
-    <!-- LINK 2 (верхнее звено, 0.30 м) -->
+    <!-- LINK 2, предплечье -->
     <link name="link_2">
         <visual>
-            <origin xyz="0 0 0.15" rpy="0 0 0"/>
-            <geometry><cylinder length="0.30" radius="0.05"/></geometry>
+            <origin xyz="0 0 ${forearm_length / 2}" rpy="0 0 0"/>
+            <geometry><cylinder length="${forearm_length}" radius="0.03"/></geometry>
             <material name="orange"/>
         </visual>
         <collision>
-            <origin xyz="0 0 0.15" rpy="0 0 0"/>
-            <geometry><cylinder length="0.30" radius="0.05"/></geometry>
-        </collision>
-        <inertial>
-            <origin xyz="0 0 0.15" rpy="0 0 0"/>
-            <mass value="1.4"/>
-            <inertia ixx="0.011375" ixy="0.0" ixz="0.0" iyy="0.011375" iyz="0.0" izz="0.00175"/>
+            <origin xyz="0 0 ${forearm_length / 2}" rpy="0 0 0"/>
+            <geometry><cylinder length="${forearm_length}" radius="0.03"/></geometry>
+        </collision>
+        <inertial>
+            <origin xyz="0 0 ${forearm_length / 2}" rpy="0 0 0"/>
+            <mass value="${forearm_mass}"/>
+            <inertia
+                ixx="${forearm_mass * (3 * 0.03 ** 2 + forearm_length ** 2) / 12}"
+                ixy="0.0" ixz="0.0"
+                iyy="${forearm_mass * (3 * 0.03 ** 2 + forearm_length ** 2) / 12}"
+                iyz="0.0"
+                izz="${forearm_mass * 0.03 ** 2 / 2}"/>
         </inertial>
     </link>
@@ -95,28 +128,33 @@
         <material>Gazebo/Orange</material>
     </gazebo>
-    <!-- JOINT 3: ELBOW PITCH (ось Y), 0.75 -> 0.95 м -->
+    <!-- JOINT 3, наклон локтя вокруг Y -->
     <joint name="joint_3" type="revolute">
         <parent link="link_2"/>
         <child link="link_3"/>
-        <origin xyz="0 0 0.30" rpy="0 0 0"/>
+        <origin xyz="0 0 ${forearm_length}" rpy="0 0 0"/>
         <axis xyz="0 1 0"/>
         <limit lower="-2.6180" upper="2.6180" effort="100.0" velocity="2.5"/>
         <dynamics damping="0.5" friction="0.1"/>
     </joint>
-    <!-- LINK 3 (предплечье, 0.20 м) -->
+    <!-- LINK 3, основание запястья -->
     <link name="link_3">
         <visual>
-            <origin xyz="0 0 0.10" rpy="0 0 0"/>
-            <geometry><cylinder length="0.20" radius="0.045"/></geometry>
+            <origin xyz="0 0 ${wrist_mount_length / 2}" rpy="0 0 0"/>
+            <geometry><cylinder length="${wrist_mount_length}" radius="0.027"/></geometry>
             <material name="green"/>
         </visual>
         <collision>
-            <origin xyz="0 0 0.10" rpy="0 0 0"/>
-            <geometry><cylinder length="0.20" radius="0.045"/></geometry>
-        </collision>
-        <inertial>
-            <origin xyz="0 0 0.10" rpy="0 0 0"/>
-            <mass value="0.9"/>
-            <inertia ixx="0.003456" ixy="0.0" ixz="0.0" iyy="0.003456" iyz="0.0" izz="0.000911"/>
+            <origin xyz="0 0 ${wrist_mount_length / 2}" rpy="0 0 0"/>
+            <geometry><cylinder length="${wrist_mount_length}" radius="0.027"/></geometry>
+        </collision>
+        <inertial>
+            <origin xyz="0 0 ${wrist_mount_length / 2}" rpy="0 0 0"/>
+            <mass value="${wrist_mount_mass}"/>
+            <inertia
+                ixx="${wrist_mount_mass * (3 * 0.027 ** 2 + wrist_mount_length ** 2) / 12}"
+                ixy="0.0" ixz="0.0"
+                iyy="${wrist_mount_mass * (3 * 0.027 ** 2 + wrist_mount_length ** 2) / 12}"
+                iyz="0.0"
+                izz="${wrist_mount_mass * 0.027 ** 2 / 2}"/>
         </inertial>
     </link>
@@ -124,28 +162,33 @@
         <material>Gazebo/Green</material>
     </gazebo>
-    <!-- JOINT 4: WRIST ROLL (ось Z) -->
+    <!-- JOINT 4, вращение запястья вокруг Z -->
     <joint name="joint_4" type="revolute">
         <parent link="link_3"/>
         <child link="link_4"/>
-        <origin xyz="0 0 0.20" rpy="0 0 0"/>
+        <origin xyz="0 0 ${wrist_mount_length}" rpy="0 0 0"/>
         <axis xyz="0 0 1"/>
         <limit lower="-3.14159" upper="3.14159" effort="50.0" velocity="3.0"/>
         <dynamics damping="0.3" friction="0.05"/>
     </joint>
-    <!-- LINK 4 (корпус кисти, 0.05 м) -->
+    <!-- LINK 4, корпус запястья -->
     <link name="link_4">
         <visual>
-            <origin xyz="0 0 0.025" rpy="0 0 0"/>
-            <geometry><cylinder length="0.05" radius="0.055"/></geometry>
+            <origin xyz="0 0 ${wrist_roll_length / 2}" rpy="0 0 0"/>
+            <geometry><cylinder length="${wrist_roll_length}" radius="0.04"/></geometry>
             <material name="red"/>
         </visual>
         <collision>
-            <origin xyz="0 0 0.025" rpy="0 0 0"/>
-            <geometry><cylinder length="0.05" radius="0.055"/></geometry>
-        </collision>
-        <inertial>
-            <origin xyz="0 0 0.025" rpy="0 0 0"/>
-            <mass value="0.4"/>
-            <inertia ixx="0.000386" ixy="0.0" ixz="0.0" iyy="0.000386" iyz="0.0" izz="0.000605"/>
+            <origin xyz="0 0 ${wrist_roll_length / 2}" rpy="0 0 0"/>
+            <geometry><cylinder length="${wrist_roll_length}" radius="0.04"/></geometry>
+        </collision>
+        <inertial>
+            <origin xyz="0 0 ${wrist_roll_length / 2}" rpy="0 0 0"/>
+            <mass value="${wrist_roll_mass}"/>
+            <inertia
+                ixx="${wrist_roll_mass * (3 * 0.04 ** 2 + wrist_roll_length ** 2) / 12}"
+                ixy="0.0" ixz="0.0"
+                iyy="${wrist_roll_mass * (3 * 0.04 ** 2 + wrist_roll_length ** 2) / 12}"
+                iyz="0.0"
+                izz="${wrist_roll_mass * 0.04 ** 2 / 2}"/>
         </inertial>
     </link>
@@ -153,28 +196,33 @@
         <material>Gazebo/Red</material>
     </gazebo>
-    <!-- JOINT 5: WRIST PITCH (ось Y) -->
+    <!-- JOINT 5, наклон запястья вокруг Y -->
     <joint name="joint_5" type="revolute">
         <parent link="link_4"/>
         <child link="link_5"/>
-        <origin xyz="0 0 0.05" rpy="0 0 0"/>
+        <origin xyz="0 0 ${wrist_roll_length}" rpy="0 0 0"/>
         <axis xyz="0 1 0"/>
         <limit lower="-2.0944" upper="2.0944" effort="50.0" velocity="3.0"/>
         <dynamics damping="0.3" friction="0.05"/>
     </joint>
-    <!-- LINK 5 (качалка кисти, 0.05 м) -->
+    <!-- LINK 5, опора фланца -->
     <link name="link_5">
         <visual>
-            <origin xyz="0 0 0.025" rpy="0 0 0"/>
-            <geometry><cylinder length="0.05" radius="0.05"/></geometry>
+            <origin xyz="0 0 ${wrist_pitch_length / 2}" rpy="0 0 0"/>
+            <geometry><cylinder length="${wrist_pitch_length}" radius="0.035"/></geometry>
             <material name="gray"/>
         </visual>
         <collision>
-            <origin xyz="0 0 0.025" rpy="0 0 0"/>
-            <geometry><cylinder length="0.05" radius="0.05"/></geometry>
-        </collision>
-        <inertial>
-            <origin xyz="0 0 0.025" rpy="0 0 0"/>
-            <mass value="0.3"/>
-            <inertia ixx="0.00025" ixy="0.0" ixz="0.0" iyy="0.00025" iyz="0.0" izz="0.000375"/>
+            <origin xyz="0 0 ${wrist_pitch_length / 2}" rpy="0 0 0"/>
+            <geometry><cylinder length="${wrist_pitch_length}" radius="0.035"/></geometry>
+        </collision>
+        <inertial>
+            <origin xyz="0 0 ${wrist_pitch_length / 2}" rpy="0 0 0"/>
+            <mass value="${wrist_pitch_mass}"/>
+            <inertia
+                ixx="${wrist_pitch_mass * (3 * 0.035 ** 2 + wrist_pitch_length ** 2) / 12}"
+                ixy="0.0" ixz="0.0"
+                iyy="${wrist_pitch_mass * (3 * 0.035 ** 2 + wrist_pitch_length ** 2) / 12}"
+                iyz="0.0"
+                izz="${wrist_pitch_mass * 0.035 ** 2 / 2}"/>
         </inertial>
     </link>
@@ -182,28 +230,33 @@
         <material>Gazebo/Grey</material>
     </gazebo>
-    <!-- JOINT 6: TOOL ROLL (ось Z) -->
+    <!-- JOINT 6, вращение фланца вокруг Z -->
     <joint name="joint_6" type="revolute">
         <parent link="link_5"/>
         <child link="link_6"/>
-        <origin xyz="0 0 0.05" rpy="0 0 0"/>
+        <origin xyz="0 0 ${wrist_pitch_length}" rpy="0 0 0"/>
         <axis xyz="0 0 1"/>
         <limit lower="-3.14159" upper="3.14159" effort="30.0" velocity="3.0"/>
         <dynamics damping="0.3" friction="0.05"/>
     </joint>
-    <!-- LINK 6 (фланец инструмента, 0.05 м) -->
+    <!-- LINK 6, фланец инструмента -->
     <link name="link_6">
         <visual>
-            <origin xyz="0 0 0.025" rpy="0 0 0"/>
-            <geometry><cylinder length="0.05" radius="0.045"/></geometry>
+            <origin xyz="0 0 ${tool_flange_length / 2}" rpy="0 0 0"/>
+            <geometry><cylinder length="${tool_flange_length}" radius="0.03"/></geometry>
             <material name="blue"/>
         </visual>
         <collision>
-            <origin xyz="0 0 0.025" rpy="0 0 0"/>
-            <geometry><cylinder length="0.05" radius="0.045"/></geometry>
-        </collision>
-        <inertial>
-            <origin xyz="0 0 0.025" rpy="0 0 0"/>
-            <mass value="0.2"/>
-            <inertia ixx="0.000143" ixy="0.0" ixz="0.0" iyy="0.000143" iyz="0.0" izz="0.000203"/>
+            <origin xyz="0 0 ${tool_flange_length / 2}" rpy="0 0 0"/>
+            <geometry><cylinder length="${tool_flange_length}" radius="0.03"/></geometry>
+        </collision>
+        <inertial>
+            <origin xyz="0 0 ${tool_flange_length / 2}" rpy="0 0 0"/>
+            <mass value="${tool_flange_mass}"/>
+            <inertia
+                ixx="${tool_flange_mass * (3 * 0.03 ** 2 + tool_flange_length ** 2) / 12}"
+                ixy="0.0" ixz="0.0"
+                iyy="${tool_flange_mass * (3 * 0.03 ** 2 + tool_flange_length ** 2) / 12}"
+                iyz="0.0"
+                izz="${tool_flange_mass * 0.03 ** 2 / 2}"/>
         </inertial>
     </link>
@@ -262,5 +315,5 @@
         <parent link="link_6"/>
         <child link="tcp"/>
-        <origin xyz="0 0 0.05" rpy="0 0 0"/>
+        <origin xyz="0 0 ${tcp_offset}" rpy="0 0 0"/>
     </joint>
 </robot>
